File: block-designs/witch-phase2a/witch-phase2a.brd (EAGLE design)
At the start: 134.6 x 100 mm, 30 parts, among them IC1 74LS73N, IC10 74LS32N, IC11 74LS157N, IC12 74LS08N, IC2 74LS73N, IC3 74LS08N, IC4 74LS08N, IC5 74LS73N, IC6 74LS73N, IC7 74LS08N, IC8 74LS08N, IC9 74LS157N

Commit message: updated board layouts
Connections:
- net CARRYOUT0: now also IC10.13; no longer IC10.5
- net CARRYOUT1: now also IC10.2; no longer IC10.10
- net CARRYOUT2: now also IC10.5; no longer IC10.13
- net CARRYOUT3: now also IC10.10; no longer IC10.2
Routing:
- net CARRYOUT1: track 123.0 -> 103.4 mm
- net COMP3: track 142.8 -> 156.8 mm, vias 1 -> 0
- net CARRYOUT3: track 152.8 -> 166.7 mm, vias 0 -> 2
- net CARRYOUT0: track 110.2 -> 97.4 mm, vias 1 -> 0
- net CARRYOUT2: track 140.0 -> 143.7 mm
Changed lines of the file:
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@@
 <?xml version="1.0" encoding="utf-8"?>
 <!DOCTYPE eagle SYSTEM "eagle.dtd">
-<eagle version="6.5.0">
+<eagle version="6.4">
 <drawing>
 <settings>
@@
 <contactref element="IC11" pad="10"/>
 <contactref element="IC9" pad="13"/>
-<via x="80.01" y="33.02" extent="1-16" drill="0.508"/>
-<wire x1="80.01" y1="33.02" x2="80.01" y2="24.13" width="0.254" layer="1"/>
-<wire x1="50.8" y1="86.36" x2="55.245" y2="86.36" width="0.254" layer="16"/>
-<wire x1="55.245" y1="86.36" x2="58.42" y2="83.185" width="0.254" layer="16"/>
-<wire x1="60.325" y1="66.675" x2="76.2" y2="66.675" width="0.254" layer="16"/>
-<wire x1="76.2" y1="66.675" x2="80.01" y2="62.865" width="0.254" layer="16"/>
-<wire x1="80.01" y1="62.865" x2="80.01" y2="33.02" width="0.254" layer="16"/>
-<wire x1="114.3" y1="54.61" x2="114.3" y2="57.15" width="0.254" layer="1"/>
-<wire x1="114.3" y1="57.15" x2="112.395" y2="59.055" width="0.254" layer="1"/>
-<wire x1="112.395" y1="59.055" x2="92.075" y2="59.055" width="0.254" layer="1"/>
-<wire x1="92.075" y1="59.055" x2="80.01" y2="46.99" width="0.254" layer="1"/>
-<wire x1="80.01" y1="46.99" x2="80.01" y2="33.02" width="0.254" layer="1"/>
-<wire x1="58.42" y1="83.185" x2="58.42" y2="68.58" width="0.254" layer="16"/>
-<wire x1="58.42" y1="68.58" x2="60.325" y2="66.675" width="0.254" layer="16"/>
+<wire x1="50.8" y1="86.36" x2="56.515" y2="86.36" width="0.254" layer="16"/>
+<wire x1="56.515" y1="86.36" x2="58.42" y2="84.455" width="0.254" layer="16"/>
+<wire x1="58.42" y1="84.455" x2="58.42" y2="69.85" width="0.254" layer="16"/>
+<wire x1="58.42" y1="69.85" x2="60.96" y2="67.31" width="0.254" layer="16"/>
+<wire x1="60.96" y1="67.31" x2="107.95" y2="67.31" width="0.254" layer="16"/>
+<wire x1="107.95" y1="67.31" x2="114.3" y2="60.96" width="0.254" layer="16"/>
+<wire x1="114.3" y1="60.96" x2="114.3" y2="54.61" width="0.254" layer="16"/>
+<wire x1="114.3" y1="54.61" x2="114.3" y2="57.785" width="0.254" layer="1"/>
+<wire x1="114.3" y1="57.785" x2="112.395" y2="59.69" width="0.254" layer="1"/>
+<wire x1="112.395" y1="59.69" x2="90.17" y2="59.69" width="0.254" layer="1"/>
+<wire x1="90.17" y1="59.69" x2="80.01" y2="49.53" width="0.254" layer="1"/>
+<wire x1="80.01" y1="49.53" x2="80.01" y2="24.13" width="0.254" layer="1"/>
 </signal>
 <signal name="ADD1">
@@
 <signal name="CARRYOUT1">
 <contactref element="IC4" pad="6"/>
-<contactref element="IC10" pad="10"/>
-<wire x1="43.18" y1="38.1" x2="38.1" y2="38.1" width="0.254" layer="1"/>
-<wire x1="38.1" y1="38.1" x2="36.195" y2="36.195" width="0.254" layer="1"/>
-<wire x1="36.195" y1="36.195" x2="36.195" y2="6.985" width="0.254" layer="1"/>
-<wire x1="36.195" y1="6.985" x2="36.83" y2="6.35" width="0.254" layer="1"/>
-<wire x1="36.83" y1="6.35" x2="80.01" y2="6.35" width="0.254" layer="1"/>
-<wire x1="80.01" y1="6.35" x2="87.63" y2="13.97" width="0.254" layer="1"/>
-<wire x1="87.63" y1="13.97" x2="87.63" y2="26.035" width="0.254" layer="1"/>
-<wire x1="87.63" y1="26.035" x2="89.535" y2="27.94" width="0.254" layer="1"/>
-<wire x1="89.535" y1="27.94" x2="101.6" y2="27.94" width="0.254" layer="1"/>
-<wire x1="101.6" y1="27.94" x2="102.87" y2="26.67" width="0.254" layer="1"/>
-<wire x1="102.87" y1="26.67" x2="102.87" y2="24.13" width="0.254" layer="1"/>
+<contactref element="IC10" pad="2"/>
+<wire x1="43.18" y1="38.1" x2="39.37" y2="38.1" width="0.254" layer="1"/>
+<wire x1="39.37" y1="38.1" x2="36.195" y2="34.925" width="0.254" layer="1"/>
+<wire x1="88.265" y1="5.08" x2="95.25" y2="12.065" width="0.254" layer="1"/>
+<wire x1="95.25" y1="12.065" x2="95.25" y2="16.51" width="0.254" layer="1"/>
+<wire x1="36.195" y1="34.925" x2="36.195" y2="6.985" width="0.254" layer="1"/>
+<wire x1="36.195" y1="6.985" x2="38.1" y2="5.08" width="0.254" layer="1"/>
+<wire x1="38.1" y1="5.08" x2="88.265" y2="5.08" width="0.254" layer="1"/>
 </signal>
 <signal name="N$2">
@@
 <signal name="CARRYOUT0">
 <contactref element="IC3" pad="3"/>
-<contactref element="IC10" pad="5"/>
-<wire x1="43.18" y1="24.13" x2="31.75" y2="24.13" width="0.254" layer="16"/>
-<via x="31.75" y="24.13" extent="1-16" drill="0.6"/>
-<wire x1="31.75" y1="24.13" x2="31.75" y2="7.62" width="0.254" layer="1"/>
-<wire x1="34.925" y1="4.445" x2="99.06" y2="4.445" width="0.254" layer="1"/>
-<wire x1="99.06" y1="4.445" x2="102.87" y2="8.255" width="0.254" layer="1"/>
-<wire x1="102.87" y1="8.255" x2="102.87" y2="16.51" width="0.254" layer="1"/>
-<wire x1="31.75" y1="7.62" x2="34.925" y2="4.445" width="0.254" layer="1"/>
+<contactref element="IC10" pad="13"/>
+<wire x1="43.18" y1="24.13" x2="38.735" y2="24.13" width="0.254" layer="1"/>
+<wire x1="38.735" y1="24.13" x2="37.465" y2="22.86" width="0.254" layer="1"/>
+<wire x1="37.465" y1="22.86" x2="37.465" y2="6.985" width="0.254" layer="1"/>
+<wire x1="37.465" y1="6.985" x2="38.735" y2="5.715" width="0.254" layer="1"/>
+<wire x1="38.735" y1="5.715" x2="79.375" y2="5.715" width="0.254" layer="1"/>
+<wire x1="79.375" y1="5.715" x2="88.9" y2="15.24" width="0.254" layer="1"/>
+<wire x1="88.9" y1="15.24" x2="88.9" y2="24.765" width="0.254" layer="1"/>
+<wire x1="88.9" y1="24.765" x2="91.44" y2="27.305" width="0.254" layer="1"/>
+<wire x1="91.44" y1="27.305" x2="93.98" y2="27.305" width="0.254" layer="1"/>
+<wire x1="93.98" y1="27.305" x2="95.25" y2="26.035" width="0.254" layer="1"/>
+<wire x1="95.25" y1="26.035" x2="95.25" y2="24.13" width="0.254" layer="1"/>
 </signal>
 <signal name="CARRYDONE0">
@@
 <signal name="CARRYOUT2">
 <contactref element="IC7" pad="3"/>
-<contactref element="IC10" pad="13"/>
-<wire x1="43.18" y1="67.31" x2="36.83" y2="67.31" width="0.254" layer="1"/>
-<wire x1="36.83" y1="67.31" x2="34.925" y2="65.405" width="0.254" layer="1"/>
-<wire x1="34.925" y1="65.405" x2="34.925" y2="6.985" width="0.254" layer="1"/>
-<wire x1="34.925" y1="6.985" x2="36.195" y2="5.715" width="0.254" layer="1"/>
-<wire x1="36.195" y1="5.715" x2="81.915" y2="5.715" width="0.254" layer="1"/>
-<wire x1="81.915" y1="5.715" x2="90.17" y2="13.97" width="0.254" layer="1"/>
-<wire x1="90.17" y1="13.97" x2="90.17" y2="18.415" width="0.254" layer="1"/>
-<wire x1="90.17" y1="18.415" x2="92.075" y2="20.32" width="0.254" layer="1"/>
-<wire x1="92.075" y1="20.32" x2="93.98" y2="20.32" width="0.254" layer="1"/>
-<wire x1="93.98" y1="20.32" x2="95.25" y2="21.59" width="0.254" layer="1"/>
-<wire x1="95.25" y1="21.59" x2="95.25" y2="24.13" width="0.254" layer="1"/>
+<contactref element="IC10" pad="5"/>
+<wire x1="43.18" y1="67.31" x2="38.1" y2="67.31" width="0.254" layer="1"/>
+<wire x1="38.1" y1="67.31" x2="34.925" y2="64.135" width="0.254" layer="1"/>
+<wire x1="34.925" y1="64.135" x2="34.925" y2="6.35" width="0.254" layer="1"/>
+<wire x1="34.925" y1="6.35" x2="36.83" y2="4.445" width="0.254" layer="1"/>
+<wire x1="36.83" y1="4.445" x2="95.25" y2="4.445" width="0.254" layer="1"/>
+<wire x1="95.25" y1="4.445" x2="102.87" y2="12.065" width="0.254" layer="1"/>
+<wire x1="102.87" y1="12.065" x2="102.87" y2="16.51" width="0.254" layer="1"/>
 </signal>
 <signal name="CARRYDONE2">
@@
 <signal name="CARRYOUT3">
 <contactref element="IC8" pad="6"/>
-<contactref element="IC10" pad="2"/>
+<contactref element="IC10" pad="10"/>
 <wire x1="43.18" y1="81.28" x2="35.56" y2="81.28" width="0.254" layer="1"/>
 <wire x1="35.56" y1="81.28" x2="33.655" y2="79.375" width="0.254" layer="1"/>
-<wire x1="33.655" y1="79.375" x2="33.655" y2="6.985" width="0.254" layer="1"/>
-<wire x1="33.655" y1="6.985" x2="35.56" y2="5.08" width="0.254" layer="1"/>
-<wire x1="35.56" y1="5.08" x2="88.9" y2="5.08" width="0.254" layer="1"/>
-<wire x1="88.9" y1="5.08" x2="95.25" y2="11.43" width="0.254" layer="1"/>
-<wire x1="95.25" y1="11.43" x2="95.25" y2="16.51" width="0.254" layer="1"/>
+<wire x1="33.655" y1="79.375" x2="33.655" y2="8.89" width="0.254" layer="1"/>
+<via x="33.655" y="8.89" extent="1-16" drill="0.6"/>
+<wire x1="33.655" y1="8.89" x2="48.895" y2="8.89" width="0.254" layer="16"/>
+<via x="48.895" y="8.89" extent="1-16" drill="0.6"/>
+<wire x1="48.895" y1="8.89" x2="80.01" y2="8.89" width="0.254" layer="1"/>
+<wire x1="80.01" y1="8.89" x2="87.63" y2="16.51" width="0.254" layer="1"/>
+<wire x1="87.63" y1="16.51" x2="87.63" y2="26.035" width="0.254" layer="1"/>
+<wire x1="102.87" y1="26.035" x2="102.87" y2="24.13" width="0.254" layer="1"/>
+<wire x1="87.63" y1="26.035" x2="90.17" y2="28.575" width="0.254" layer="1"/>
+<wire x1="90.17" y1="28.575" x2="100.33" y2="28.575" width="0.254" layer="1"/>
+<wire x1="100.33" y1="28.575" x2="102.87" y2="26.035" width="0.254" layer="1"/>
 </signal>
 <signal name="CARRYDONE3">
