File: block-designs/witch-phase2a/witch-phase2a.sch (EAGLE design)
At the start: 13 parts, among them IC1 74LS73D, IC10 74LS08D, IC11 74LS157D, IC2 74LS08D, IC4 74LS157D, IC5 74LS73D, IC6 74LS08D, IC7 74LS73D, IC8 74LS08D, IC9 74LS73D

Commit message: added base schematic
Parts:
- removed JP5, JP9: (no value), pinhead:PINHD-2X10
- added IC3: 74ALS08D, 74xx-us:74ALS08D
- added JP2, JP3: (no value), pinhead:PINHD-2X10
Connections:
- removed net CARRY0: IC1A.CLK
- removed net CARRY1: IC5A.CLK
- removed net CARRY2: IC7A.CLK
- removed net CARRY3: IC9A.CLK
- removed net ZC0: IC1B.CLK
- removed net ZC1: IC5B.CLK
- removed net ZC2: IC7B.CLK
- removed net ZC3: IC9B.CLK
- new net CARRY_COMPLETE: IC3C.O, JP3.16
- new net DK_RESET: JP1.3, JP2.3
- new net N$17: IC4A.4Y, JP1.17
- new net N$18: IC4A.3Y, JP1.13
- new net N$19: IC4A.2Y, JP1.9
- new net N$20: IC4A.1Y, JP1.5
- new net N$21: IC11A.4Y, JP2.17
- new net N$22: IC11A.3Y, JP2.13
- new net N$23: IC11A.2Y, JP2.9
- new net N$24: IC11A.1Y, JP2.5
- new net N$25: IC3A.O, IC3C.I0
- new net N$26: IC3B.O, IC3C.I1
- new net ZCR0: IC1A.CLK, JP2.6
- new net ZCR1: IC5A.CLK, JP2.10
- new net ZCR2: IC7A.CLK, JP2.14
- new net ZCR3: IC9A.CLK, JP2.18
- new net ZCS0: IC1B.CLK, JP1.6
- new net ZCS1: IC5B.CLK, JP1.10
- new net ZCS2: IC7B.CLK, JP1.14
- new net ZCS3: IC9B.CLK, JP1.18
- net 10A_PULSES: now also JP1.4, JP2.4, JP3.4
- net CARRYDONE0: now also IC3A.I0
- net CARRYDONE1: now also IC3A.I1
- net CARRYDONE2: now also IC3B.I0
- net CARRYDONE3: now also IC3B.I1
- net CARRY_PULSES: now also JP3.12
- net GND: now also JP1.19, JP1.20, JP2.19, JP2.20, JP3.19, JP3.20
- net RESET: now also JP3.3
- net TRANSFER_PULSES: now also JP3.8
- net VCC: now also JP1.1, JP1.2, JP2.1, JP2.2, JP3.1, JP3.2

Commit message: routed and updated transferboard and add dekatron board
Parts:
- added C1, C10, C11, C12, C2, C3, C4, C5, C6, C7, C8, C9: (no value), resistor:C-US025-025X050
- added C13, C14, C15: (no value), resistor:CPOL-USE2-5
- added IC12: 74LS08N, 74xx-us:74LS08N
- IC1, IC5: value 74LS73D -> 74LS73N; device 74xx-us:74LS73D -> 74xx-us:74LS73N
- IC10: value 74LS08D -> 74LS32N; device 74xx-us:74LS08D -> 74xx-us:74LS32N
- IC11: value 74LS157D -> 74LS157N; device 74xx-us:74LS157D -> 74xx-us:74LS157N
- IC2, IC6: value 74LS08D -> 74LS73N; device 74xx-us:74LS08D -> 74xx-us:74LS73N
- IC3: value 74ALS08D -> 74LS08N; device 74xx-us:74ALS08D -> 74xx-us:74LS08N
- IC4: value 74LS157D -> 74LS08N; device 74xx-us:74LS157D -> 74xx-us:74LS08N
- IC7: value 74LS73D -> 74LS08N; device 74xx-us:74LS73D -> 74xx-us:74LS08N
- IC8: value 74LS08D -> 74LS08N; device 74xx-us:74LS08D -> 74xx-us:74LS08N
- IC9: value 74LS73D -> 74LS157N; device 74xx-us:74LS73D -> 74xx-us:74LS157N
Connections:
- removed net DK_RESET: JP1.3, JP2.3
- removed net N$17: IC4A.4Y, JP1.17
- removed net N$18: IC4A.3Y, JP1.13
- removed net N$19: IC4A.2Y, JP1.9
- removed net N$20: IC4A.1Y, JP1.5
- removed net N$21: IC11A.4Y, JP2.17
- removed net N$22: IC11A.3Y, JP2.13
- removed net N$23: IC11A.2Y, JP2.9
- removed net N$24: IC11A.1Y, JP2.5
- new net DKR0: IC10A.O, JP2.17
- new net DKR1: IC10B.O, JP2.13
- new net DKR2: IC10C.O, JP2.9
- new net DKR3: IC10D.O, JP2.5
- new net DKS0: IC9A.1Y, JP1.17
- new net DKS1: IC9A.2Y, JP1.13
- new net DKS2: IC9A.3Y, JP1.9
- new net DKS3: IC9A.4Y, JP1.5
- new net TRANSFEROUT0: IC10A.I0, IC11A.2Y
- new net TRANSFEROUT1: IC10B.I0, IC11A.1Y
- new net TRANSFEROUT2: IC10C.I0, IC11A.4Y
- new net TRANSFEROUT3: IC10D.I0, IC11A.3Y
- net 10A_PULSES: now also IC9A.1A, IC9A.2A, IC9A.3A, IC9A.4A; no longer IC4A.1A, IC4A.2A, IC4A.3A, IC4A.4A
- net ADD0: now also IC11A.2A, IC3D.O; no longer IC11A.1A, IC2C.O
- net ADD1: now also IC11A.1A, IC4C.O; no longer IC11A.2A, IC6C.O
- net ADD2: now also IC11A.4A, IC7D.O; no longer IC11A.3A, IC8C.O
- net ADD3: now also IC11A.3A, IC8C.O; no longer IC10C.O, IC11A.4A
- net CARRYDONE0: now also IC12A.I0, IC3B.O; no longer IC2A.O, IC3A.I0
- net CARRYDONE1: now also IC12A.I1, IC4A.O; no longer IC3A.I1, IC6A.O
- net CARRYDONE2: now also IC12B.I0, IC7B.O; no longer IC3B.I0, IC8A.O
- net CARRYDONE3: now also IC12B.I1, IC8A.O; no longer IC10A.O, IC3B.I1
- net CARRYOUT0: now also IC10B.I1, IC3A.O; no longer IC2B.O
- net CARRYOUT1: now also IC10C.I1, IC4B.O; no longer IC6B.O
- net CARRYOUT2: now also IC10D.I1, IC7A.O; no longer IC8B.O
- net CARRYOUT3: now also IC10A.I1, IC8B.O; no longer IC10B.O
- net CARRY_COMPLETE: now also IC12C.O; no longer IC3C.O
- net CARRY_PULSES: now also IC3A.I0, IC3B.I0, IC4A.I0, IC4B.I0, IC7A.I0, IC7B.I0, IC8B.I0; no longer IC10A.I0, IC10B.I1, IC2A.I0, IC2B.I1, IC6A.I0, IC6B.I1, IC8B.I1
- net COMP0: now also IC11A.2B, IC3C.O, IC9A.1B; no longer IC11A.1B, IC2D.O, IC4A.1B
- net COMP1: now also IC11A.1B, IC4D.O, IC9A.2B; no longer IC11A.2B, IC4A.2B, IC6D.O
- net COMP2: now also IC11A.4B, IC7C.O, IC9A.3B; no longer IC11A.3B, IC4A.3B, IC8D.O
- net COMP3: now also IC11A.3B, IC8D.O, IC9A.4B; no longer IC10D.O, IC11A.4B, IC4A.4B
- net GND: now also C1.2, C10.2, C11.2, C12.2, C13.-, C14.-, C15.-, C2.2, C3.2, C4.2, C5.2, C6.2, C7.2, C8.2, C9.2, IC10P.GND, IC11P.GND, IC12P.GND, IC1P.GND, IC2A.K, IC2B.K, IC2P.GND, IC3P.GND, IC4P.GND, IC5P.GND, IC6A.K, IC6B.K, IC6P.GND, IC7P.GND, IC8P.GND, IC9P.GND; no longer IC7A.K, IC7B.K, IC9A.K, IC9B.K
- net N$1: now also IC2B.Q, IC3A.I1; no longer IC1A.Q, IC2B.I0
- net N$10: now also IC5A.!Q, IC7C.I1; no longer IC7A.!Q, IC8A.I1
- net N$11: now also IC5A.Q, IC7D.I1; no longer IC7B.Q, IC8C.I1
- net N$12: now also IC6B.Q, IC7A.I1; no longer IC7B.!Q, IC8D.I0
- net N$13: now also IC6A.!Q, IC8A.I1; no longer IC10B.I0, IC9A.Q
- net N$14: now also IC5B.!Q, IC8D.I1; no longer IC10A.I1, IC9A.!Q
- net N$15: now also IC5B.Q, IC8C.I1; no longer IC10C.I1, IC9B.Q
- net N$16: now also IC6A.Q, IC8B.I1; no longer IC10D.I0, IC9B.!Q
- net N$2: now also IC2B.!Q, IC3B.I1; no longer IC1A.!Q, IC2A.I1
- net N$25: now also IC12A.O, IC12C.I1; no longer IC3A.O, IC3C.I0
- net N$26: now also IC12B.O, IC12C.I0; no longer IC3B.O, IC3C.I1
- net N$3: now also IC2A.Q, IC4B.I1; no longer IC5A.Q, IC6B.I0
- net N$4: now also IC1A.Q, IC3D.I1; no longer IC1B.Q, IC2C.I1
- net N$5: now also IC1A.!Q, IC3C.I1; no longer IC1B.!Q, IC2D.I0
- net N$6: now also IC2A.!Q, IC4A.I1; no longer IC5A.!Q, IC6A.I1
- net N$7: now also IC1B.!Q, IC4D.I1; no longer IC5B.Q, IC6C.I1
- net N$8: now also IC1B.Q, IC4C.I1; no longer IC5B.!Q, IC6D.I0
- net N$9: now also IC6B.!Q, IC7B.I1; no longer IC7A.Q, IC8B.I0
- net RESET: now also IC2A.CL, IC2B.CL, IC6A.CL, IC6B.CL; no longer IC7A.CL, IC7B.CL, IC9A.CL, IC9B.CL
- net TRANSFER_PULSES: now also IC3C.I0, IC3D.I0, IC4C.I0, IC4D.I0, IC7C.I0, IC7D.I0, IC8D.I0; no longer IC10C.I0, IC10D.I1, IC2C.I0, IC2D.I1, IC6C.I0, IC6D.I1, IC8D.I1
- net VCC: now also C1.1, C10.1, C11.1, C12.1, C13.+, C14.+, C15.+, C2.1, C3.1, C4.1, C5.1, C6.1, C7.1, C8.1, C9.1, IC10P.VCC, IC11P.VCC, IC12P.VCC, IC1P.VCC, IC2A.J, IC2B.J, IC2P.VCC, IC3P.VCC, IC4P.VCC, IC5P.VCC, IC6A.J, IC6B.J, IC6P.VCC, IC7P.VCC, IC8P.VCC, IC9P.VCC; no longer IC7A.J, IC7B.J, IC9A.J, IC9B.J
- net ZCR0: now also IC2B.CLK, JP2.18; no longer IC1A.CLK, JP2.6
- net ZCR1: now also IC2A.CLK, JP2.14; no longer IC5A.CLK, JP2.10
- net ZCR2: now also IC6B.CLK, JP2.10; no longer IC7A.CLK, JP2.14
- net ZCR3: now also IC6A.CLK, JP2.6; no longer IC9A.CLK, JP2.18
- net ZCS0: now also IC1A.CLK, JP1.18; no longer IC1B.CLK, JP1.6
- net ZCS1: now also IC1B.CLK, JP1.14; no longer IC5B.CLK, JP1.10
- net ZCS2: now also IC5A.CLK, JP1.10; no longer IC7B.CLK, JP1.14
- net ZCS3: now also IC5B.CLK, JP1.6; no longer IC9B.CLK, JP1.18

Commit message: updated layouts
Connections:
- net 10A_PULSES: no longer JP1.4, JP2.4
Changed lines of the file:
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@@
 <?xml version="1.0" encoding="utf-8"?>
 <!DOCTYPE eagle SYSTEM "eagle.dtd">
-<eagle version="6.4">
+<eagle version="6.5.0">
 <drawing>
 <settings>
@@
 <pinref part="IC9" gate="A" pin="4A"/>
 </segment>
-<segment>
-<wire x1="172.72" y1="172.72" x2="203.2" y2="172.72" width="0.1524" layer="91"/>
-<label x="187.96" y="172.72" size="1.778" layer="95"/>
-<pinref part="JP1" gate="A" pin="4"/>
-</segment>
 </net>
 <net name="VCC" class="0">
@@
 </segment>
 </net>
-<net name="10A_PULSES" class="0">
-<segment>
-<pinref part="JP2" gate="A" pin="4"/>
-<wire x1="182.88" y1="134.62" x2="213.36" y2="134.62" width="0.1524" layer="91"/>
-<label x="198.12" y="134.62" size="1.778" layer="95"/>
-</segment>
-</net>

Commit message: updated board layouts
Connections:
- net CARRYOUT0: now also IC10D.I1; no longer IC10B.I1
- net CARRYOUT1: now also IC10A.I1; no longer IC10C.I1
- net CARRYOUT2: now also IC10B.I1; no longer IC10D.I1
- net CARRYOUT3: now also IC10C.I1; no longer IC10A.I1
Changed lines of the file:
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@@
 <?xml version="1.0" encoding="utf-8"?>
 <!DOCTYPE eagle SYSTEM "eagle.dtd">
-<eagle version="6.5.0">
+<eagle version="6.4">
 <drawing>
 <settings>
@@
 <net name="CARRYOUT3" class="0">
 <segment>
+<pinref part="IC10" gate="C" pin="I1"/>
+<wire x1="63.5" y1="147.32" x2="35.56" y2="147.32" width="0.1524" layer="91"/>
+<label x="35.56" y="147.32" size="1.778" layer="95"/>
+</segment>
+</net>
+<net name="CARRYOUT0" class="0">
+<segment>
+<pinref part="IC10" gate="D" pin="I1"/>
+<wire x1="63.5" y1="134.62" x2="35.56" y2="134.62" width="0.1524" layer="91"/>
+<label x="35.56" y="134.62" size="1.778" layer="95"/>
+</segment>
+</net>
+<net name="CARRYOUT2" class="0">
+<segment>
+<pinref part="IC10" gate="B" pin="I1"/>
+<wire x1="63.5" y1="160.02" x2="35.56" y2="160.02" width="0.1524" layer="91"/>
+<label x="35.56" y="160.02" size="1.778" layer="95"/>
+</segment>
+</net>
+<net name="CARRYOUT1" class="0">
+<segment>
 <pinref part="IC10" gate="A" pin="I1"/>
 <wire x1="63.5" y1="172.72" x2="35.56" y2="172.72" width="0.1524" layer="91"/>
@@
 </segment>
 </net>
-<net name="CARRYOUT0" class="0">
-<segment>
-<pinref part="IC10" gate="B" pin="I1"/>
-<wire x1="63.5" y1="160.02" x2="35.56" y2="160.02" width="0.1524" layer="91"/>
-<label x="35.56" y="160.02" size="1.778" layer="95"/>
-</segment>
-</net>
-<net name="CARRYOUT1" class="0">
-<segment>
-<pinref part="IC10" gate="C" pin="I1"/>
-<wire x1="63.5" y1="147.32" x2="35.56" y2="147.32" width="0.1524" layer="91"/>
-<label x="35.56" y="147.32" size="1.778" layer="95"/>
-</segment>
-</net>
-<net name="CARRYOUT2" class="0">
-<segment>
-<pinref part="IC10" gate="D" pin="I1"/>
-<wire x1="63.5" y1="134.62" x2="35.56" y2="134.62" width="0.1524" layer="91"/>
-<label x="35.56" y="134.62" size="1.778" layer="95"/>
-</segment>
-</net>
