File: block-designs/witch-phase2b/witch-phase2b.sch (EAGLE design)
At the start: 61 parts, among them IC1 74HC160N, IC10 74LS73N, IC11 74LS08N, IC12 74LS32N, IC2 4511N, IC3 74HC160N, IC4 4511N, IC5 74HC160N, IC6 4511N, IC7 74HC160N, IC8 4511N, IC9 74LS73N

Commit message: updated layouts
Parts:
- added R33, R34, R35, R36: (no value), resistor:R-US_0204/5
- added S1, S2, S3, S4: (no value), SparkFun-Electromechanical:TAC_SWITCHPTH
- C12, C3, C6, C9: device resistor:CPOL-USE2-5 -> resistor:C-US025-025X050
Connections:
- removed net N$28: IC3A.RCO, R16.2
- removed net N$29: IC3A.CLR
- removed net N$49: IC5A.CLK
- removed net N$50: IC5A.RCO, R24.2
- removed net N$51: IC5A.CLR
- removed net N$71: IC7A.CLK
- removed net N$72: IC7A.RCO, R32.2
- removed net N$73: IC7A.CLR
- removed net VDD: C1.1, C10.1, C11.1, C12.+, C2.1, C3.+, C4.1, C5.1, C6.+, C7.1, C8.1, C9.+, IC1A.ENP, IC1A.ENT, IC1A.LD, IC1P.VCC, IC2A.BI, IC2A.LT, IC2P.VDD, IC3A.ENP, IC3A.ENT, IC3A.LD, IC3P.VCC, IC4A.BI, IC4A.LT, IC4P.VDD, IC5A.ENP, IC5A.ENT, IC5A.LD, IC5P.VCC, IC6A.BI, IC6A.LT, IC6P.VDD, IC7A.ENP, IC7A.ENT, IC7A.LD, IC7P.VCC, IC8A.BI, IC8A.LT, IC8P.VDD
- removed net VSS: C1.2, C10.2, C11.2, C12.-, C2.2, C3.-, C4.2, C5.2, C6.-, C7.2, C8.2, C9.-, IC1P.GND, IC2A.LE, IC2P.VSS, IC3P.GND, IC4A.LE, IC4P.VSS, IC5P.GND, IC6A.LE, IC6P.VSS, IC7P.GND, IC8A.LE, IC8P.VSS, LED1.COM@1, LED1.COM@2, LED2.COM@1, LED2.COM@2, LED3.COM@1, LED3.COM@2, LED4.COM@1, LED4.COM@2
- new net BUTTON0: C3.2, IC12C.I1, R33.2, S1.3, S1.4
- new net BUTTON1: C6.2, IC12D.I1, R34.2, S2.3, S2.4
- new net BUTTON2: C9.2, IC12A.I1, R35.2, S3.3, S3.4
- new net BUTTON3: C12.2, IC12B.I1, R36.2, S4.3, S4.4
- new net DK0: IC12C.O, IC1A.CLK
- new net DK1: IC12D.O, IC3A.CLK
- new net DK2: IC12A.O, IC5A.CLK
- new net DK3: IC12B.O, IC7A.CLK
- new net DKIN0: IC12C.I0, JP1.17
- new net DKIN1: IC12D.I0, JP1.13
- new net DKIN2: IC12A.I0, JP1.9
- new net DKIN3: IC12B.I0, JP1.5
- new net DKRESET: IC10A.CL, IC10B.CL, IC9A.CL, IC9B.CL, JP1.3
- new net GND: C1.2, C10.2, C11.2, C2.2, C4.2, C5.2, C7.2, C8.2, IC10A.K, IC10B.K, IC1P.GND, IC2A.LE, IC2P.VSS, IC3P.GND, IC4A.LE, IC4P.VSS, IC5P.GND, IC6A.LE, IC6P.VSS, IC7P.GND, IC8A.LE, IC8P.VSS, IC9A.K, IC9B.K, JP1.19, JP1.20, LED1.COM@1, LED1.COM@2, LED2.COM@1, LED2.COM@2, LED3.COM@1, LED3.COM@2, LED4.COM@1, LED4.COM@2, R33.1, R34.1, R35.1, R36.1
- new net PULSES: IC11A.I0, IC11B.I0, IC11C.I0, IC11D.I0, JP1.4
- new net RESET: IC1A.CLR, IC3A.CLR, IC5A.CLR, IC7A.CLR
- new net VCC: C1.1, C10.1, C11.1, C2.1, C3.1, C4.1, C5.1, C7.1, C8.1, IC10A.J, IC10B.J, IC1A.ENP, IC1A.ENT, IC1A.LD, IC1P.VCC, IC2A.BI, IC2A.LT, IC2P.VDD, IC3A.ENP, IC3A.ENT, IC3A.LD, IC3P.VCC, IC4A.BI, IC4A.LT, IC4P.VDD, IC5A.ENP, IC5A.ENT, IC5A.LD, IC5P.VCC, IC6A.BI, IC6A.LT, IC6P.VDD, IC7A.ENP, IC7A.ENT, IC7A.LD, IC7P.VCC, IC8A.BI, IC8A.LT, IC8P.VDD, IC9A.J, IC9B.J, JP1.1, JP1.2, S1.1, S1.2, S2.1, S2.2, S3.1, S3.2, S4.1, S4.2
- new net VCC1: C6.1
- new net VCC2: C9.1
- new net VCC3: C12.1
- new net ZC0: IC10B.CLK, IC1A.RCO, R8.2
- new net ZC1: IC10A.CLK, IC3A.RCO, R16.2
- new net ZC2: IC5A.RCO, IC9B.CLK, R24.2
- new net ZC3: IC7A.RCO, IC9A.CLK, R32.2
- new net ZCOUT0: IC11D.O, JP1.18
- new net ZCOUT1: IC11C.O, JP1.14
- new net ZCOUT2: IC11B.O, JP1.10
- new net ZCOUT3: IC11A.O, JP1.6
- net N$1: now also IC11A.I1, IC9A.Q; no longer IC1A.RCO, R8.2
- net N$2: now also IC11B.I1, IC9B.Q; no longer IC1A.CLR
- net N$25: now also IC10A.Q, IC11C.I1; no longer IC1A.CLK
- net N$27: now also IC10B.Q, IC11D.I1; no longer IC3A.CLK
Other:
- note removed: "CLEAR"
- note removed: "PULSE INPUT"
- note removed: "ZC"

Commit message: updated board layouts
Parts:
- added C13, C14, C15, C16: (no value), resistor:C-US025-025X050
- added C17: (no value), resistor:CPOL-USE2-5
- added C18: (no value), resistor:C-US025-040X050
- added R37: (no value), resistor:R-US_0204/5
Connections:
- new net VDD: R37.1
- new net VSS: C18.2
- net GND: now also C13.2, C14.2, C15.2, C16.2, C17.-, IC10P.GND, IC11P.GND, IC12P.GND, IC9P.GND
- net RESET: now also C18.1, R37.2
- net VCC: now also C13.1, C14.1, C15.1, C16.1, C17.+, IC10P.VCC, IC11P.VCC, IC12P.VCC, IC9P.VCC
