File: block-designs/witch-phase2/tester-debug/keyboard-tester/keyboard-tester.brd (EAGLE design)
At the start: 99.1 x 78.7 mm, 46 parts, among them IC1 74LVC1G17DBV, IC2 74LVC1G17DBV, IC3 74LVC1G17DBV, IC4 74LVC1G17DBV, IC5 74LVC1G17DBV, IC6 74LVC1G17DBV, IC7 74LVC1G17DBV, IC8 74LVC1G17DBV, IC9 74LVC1G17DBV

Commit message: move keyboard tester to new directory for test and debug boards
Parts:
- C1: value (none) -> 10uF
- R1: value (none) -> 100k
- R6: value (none) -> 10k
Changed lines of the file:
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@@
 <?xml version="1.0" encoding="utf-8"?>
 <!DOCTYPE eagle SYSTEM "eagle.dtd">
-<eagle version="7.3.0">
+<eagle version="7.6.0">
 <drawing>
 <settings>
@@
 </element>
 <element name="S1" library="SparkFun-Electromechanical" package="TACTILE-PTH" value="" x="13.2588" y="43.2308" rot="R270"/>
-<element name="C1" library="resistor" package="C0805" value="" x="14.5796" y="51.435"/>
-<element name="R6" library="resistor" package="R0805" value="" x="9.9822" y="51.435"/>
-<element name="R1" library="resistor" package="R0805" value="" x="9.0424" y="56.4642" rot="R90"/>
+<element name="C1" library="resistor" package="C0805" value="10uF" x="14.5796" y="51.435"/>
+<element name="R6" library="resistor" package="R0805" value="10k" x="9.9822" y="51.435"/>
+<element name="R1" library="resistor" package="R0805" value="100k" x="9.0424" y="56.4642" rot="R90"/>
 <element name="IC1" library="74xx-little-us" package="SOT23-5" value="74LVC1G17DBV" x="12.9032" y="62.8396"/>
 <element name="S2" library="SparkFun-Electromechanical" package="TACTILE-PTH" value="" x="32.1818" y="43.2308" rot="R270"/>
