File: block-designs/witch-phase2/input-sequence/input-sequence.sch (EAGLE design)
At the start: 21 parts, among them IC1 74AHC1G08DBV, IC10 741G175, IC11 741G175, IC12 741G175, IC13 74AHC1G32DBV, IC14 74AHC1G32DBV, IC15 74AHC1G32DBV, IC16 74AHC1G32DBV, IC17 74AHC1G32DBV, IC18 74AHC1G32DBV, IC19 4017D, IC2 74AHC1G08DBV, IC3 74AHC1G08DBV, IC4 74AHC1G08DBV, IC5 74AHC1G08DBV, IC6 74AHC1G08DBV, IC7 741G175, IC8 741G175, IC9 741G175

Commit message: reduce pcb size, add caps, add LEDs
Parts:
- added C1, C10, C11, C12, C13, C14, C15, C16, C17, C18, C19, C2, C20, C3, C4, C5, C6, C7, C8, C9: 0.1uF, resistor:C-USC0603
- added LED1, LED2, LED3, LED4, LED5, LED6, LED7: RED, led:LEDCHIP-LED0805
- added R1: (no value), resistor:R-US_R0805
- IC1: value 74AHC1G08DBV -> 4017D; device 74xx-little-us:74AHC1G08DBV -> 40xx:4017D
- IC13: value 74AHC1G32DBV -> 741G175; device 74xx-little-us:74AHC1G32DBV -> witch-e:741G175
- IC14, IC15, IC16, IC17, IC18: value 74AHC1G32DBV -> 74AHC1G08DBV; device 74xx-little-us:74AHC1G32DBV -> 74xx-little-us:74AHC1G08DBV
- IC19: value 4017D -> 74AHC1G08DBV; device 40xx:4017D -> 74xx-little-us:74AHC1G08DBV
- IC2, IC3, IC4, IC5, IC6: value 74AHC1G08DBV -> 74AHC1G32DBV; device 74xx-little-us:74AHC1G08DBV -> 74xx-little-us:74AHC1G32DBV
- IC7: value 741G175 -> 74AHC1G32DBV; device witch-e:741G175 -> 74xx-little-us:74AHC1G32DBV
Connections:
- new net LED_SINK: LED1.C, LED2.C, LED3.C, LED4.C, LED5.C, LED6.C, LED7.C, R1.2
- net !MCLK: now also IC14A.I0, IC15A.I0, IC16A.I0, IC17A.I0, IC18A.I0, IC19A.I0; no longer IC1A.I0, IC2A.I0, IC3A.I0, IC4A.I0, IC5A.I0, IC6A.I0
- net !RESET: now also IC13G$1.!CLR, IC1A.RES; no longer IC19A.RES, IC7G$1.!CLR
- net GND: now also C1.2, C10.2, C11.2, C12.2, C13.2, C14.2, C15.2, C16.2, C17.2, C18.2, C19.2, C2.2, C20.2, C3.2, C4.2, C5.2, C6.2, C7.2, C8.2, C9.2, IC1A.ENA, IC1P.VSS, IC2A.I0, R1.1; no longer IC13A.I0, IC19A.ENA
- net N$1: now also IC15A.O, IC9G$1.CLK; no longer IC2A.O, IC8G$1.CLK
- net N$2: now also IC14A.O, IC8G$1.CLK; no longer IC1A.O, IC7G$1.CLK
- net N$3: now also IC10G$1.CLK, IC16A.O; no longer IC3A.O, IC9G$1.CLK
- net N$4: now also IC11G$1.CLK, IC17A.O; no longer IC10G$1.CLK, IC4A.O
- net N$5: now also IC12G$1.CLK, IC18A.O; no longer IC11G$1.CLK, IC5A.O
- net N$6: now also IC13G$1.CLK, IC19A.O; no longer IC12G$1.CLK, IC6A.O
- net NEXT1: now also IC2A.O, IC3A.I0; no longer IC13A.O, IC14A.I0
- net NEXT2: now also IC3A.O, IC4A.I0; no longer IC14A.O, IC15A.I0
- net NEXT3: now also IC4A.O, IC5A.I0; no longer IC15A.O, IC16A.I0
- net NEXT4: now also IC5A.O, IC6A.I0; no longer IC16A.O, IC17A.I0
- net NEXT5: now also IC6A.O, IC7A.I0; no longer IC17A.O, IC18A.I0
- net NEXT6: now also IC1A.CLK, IC7A.O; no longer IC18A.O, IC19A.CLK
- net SEQ1: now also IC1A.Q0, IC8G$1.D, LED2.A; no longer IC19A.Q0, IC7G$1.D
- net SEQ2: now also IC1A.Q1, IC9G$1.D, LED3.A; no longer IC19A.Q1, IC8G$1.D
- net SEQ3: now also IC10G$1.D, IC1A.Q2, LED4.A; no longer IC19A.Q2, IC9G$1.D
- net SEQ4: now also IC11G$1.D, IC1A.Q3, LED5.A; no longer IC10G$1.D, IC19A.Q3
- net SEQ5: now also IC12G$1.D, IC1A.Q4, LED6.A; no longer IC11G$1.D, IC19A.Q4
- net SEQ6: now also IC13G$1.D, IC1A.Q5, LED7.A; no longer IC12G$1.D, IC19A.Q5
- net SEQ7: now also IC1A.Q6, LED1.A; no longer IC19A.Q6
- net STEP1: now also IC2A.I1, IC8G$1.Q; no longer IC13A.I1, IC7G$1.Q
- net STEP2: now also IC3A.I1, IC9G$1.Q; no longer IC14A.I1, IC8G$1.Q
- net STEP3: now also IC10G$1.Q, IC4A.I1; no longer IC15A.I1, IC9G$1.Q
- net STEP4: now also IC11G$1.Q, IC5A.I1; no longer IC10G$1.Q, IC16A.I1
- net STEP5: now also IC12G$1.Q, IC6A.I1; no longer IC11G$1.Q, IC17A.I1
- net STEP6: now also IC13G$1.Q, IC7A.I1; no longer IC12G$1.Q, IC18A.I1
- net VAL1: now also IC14A.I1; no longer IC1A.I1
- net VAL2: now also IC15A.I1; no longer IC2A.I1
- net VAL3: now also IC16A.I1; no longer IC3A.I1
- net VAL4: now also IC17A.I1; no longer IC4A.I1
- net VAL5: now also IC18A.I1; no longer IC5A.I1
- net VAL6: now also IC19A.I1; no longer IC6A.I1
- net VCC: now also C1.1, C10.1, C11.1, C12.1, C13.1, C14.1, C15.1, C16.1, C17.1, C18.1, C19.1, C2.1, C20.1, C3.1, C4.1, C5.1, C6.1, C7.1, C8.1, C9.1, IC1P.VDD
Other:
- moved on the sheet: IC10, IC11, IC12, IC8, IC9, JP1, JP2

Commit message: updated layout and added inverter for reset signals
Parts:
- added IC20, IC21: 74LVC1G14DBV, 74xx-little-us:74LVC1G14DBV
- added JP3, JP4, JP5, JP6, JP7: (no value), custom-pinhead:PINHD-1X4
- added R2: (no value), resistor:R-US_R0805
- IC1: value 4017D -> 74AHC1G08DBV; device 40xx:4017D -> 74xx-little-us:74AHC1G08DBV
- IC13: value 741G175 -> 74AHC1G32DBV; device witch-e:741G175 -> 74xx-little-us:74AHC1G32DBV
- IC14, IC15, IC16, IC17, IC18: value 74AHC1G08DBV -> 74AHC1G32DBV; device 74xx-little-us:74AHC1G08DBV -> 74xx-little-us:74AHC1G32DBV
- IC19: value 74AHC1G08DBV -> 4017D; device 74xx-little-us:74AHC1G08DBV -> 40xx:4017D
- IC2, IC3, IC4, IC5, IC6: value 74AHC1G32DBV -> 74AHC1G08DBV; device 74xx-little-us:74AHC1G32DBV -> 74xx-little-us:74AHC1G08DBV
- IC7: value 74AHC1G32DBV -> 741G175; device 74xx-little-us:74AHC1G32DBV -> witch-e:741G175
- JP1, JP2: device pinhead:PINHD-1X10 -> custom-pinhead:PINHD-1X4
Connections:
- removed net SEQ1: IC1A.Q0, IC8G$1.D, JP1.2, LED2.A
- removed net SEQ2: IC1A.Q1, IC9G$1.D, JP1.3, LED3.A
- removed net SEQ3: IC10G$1.D, IC1A.Q2, JP1.4, LED4.A
- removed net SEQ4: IC11G$1.D, IC1A.Q3, JP1.5, LED5.A
- removed net SEQ5: IC12G$1.D, IC1A.Q4, JP1.6, LED6.A
- removed net SEQ6: IC13G$1.D, IC1A.Q5, JP1.7, LED7.A
- removed net SEQ7: IC1A.Q6, JP1.8, LED1.A
- new net !CLEAR: IC21A.I, JP7.2
- new net RESET: IC19A.RES, IC20A.I, IC21A.O, R2.2
- new net SEL1: IC19A.Q0, IC7G$1.D, JP1.3, LED1.A
- new net SEL2: IC19A.Q1, IC8G$1.D, JP2.3, LED2.A
- new net SEL3: IC19A.Q2, IC9G$1.D, JP3.3, LED3.A
- new net SEL4: IC10G$1.D, IC19A.Q3, JP4.3, LED4.A
- new net SEL5: IC11G$1.D, IC19A.Q4, JP5.3, LED5.A
- new net SEL6: IC12G$1.D, IC19A.Q5, JP6.3, LED6.A
- new net SEL7: IC19A.Q6, LED7.A
- net !MCLK: now also IC1A.I0, IC2A.I0, IC3A.I0, IC4A.I0, IC5A.I0, IC6A.I0, JP7.3; no longer IC14A.I0, IC15A.I0, IC16A.I0, IC17A.I0, IC18A.I0, IC19A.I0, JP2.9
- net !RESET: now also IC20A.O, IC7G$1.!CLR; no longer IC13G$1.!CLR, IC1A.RES, JP1.9
- net GND: now also IC13A.I0, IC19A.ENA, IC19P.VSS, JP1.4, JP2.4, JP3.4, JP4.4, JP5.4, JP6.4, JP7.4, R2.1; no longer IC1A.ENA, IC1P.VSS, IC2A.I0, JP1.10, JP2.10
- net N$1: now also IC2A.O, IC8G$1.CLK; no longer IC15A.O, IC9G$1.CLK
- net N$2: now also IC1A.O, IC7G$1.CLK; no longer IC14A.O, IC8G$1.CLK
- net N$3: now also IC3A.O, IC9G$1.CLK; no longer IC10G$1.CLK, IC16A.O
- net N$4: now also IC10G$1.CLK, IC4A.O; no longer IC11G$1.CLK, IC17A.O
- net N$5: now also IC11G$1.CLK, IC5A.O; no longer IC12G$1.CLK, IC18A.O
- net N$6: now also IC12G$1.CLK, IC6A.O; no longer IC13G$1.CLK, IC19A.O
- net NEXT1: now also IC13A.O, IC14A.I0; no longer IC2A.O, IC3A.I0
- net NEXT2: now also IC14A.O, IC15A.I0; no longer IC3A.O, IC4A.I0
- net NEXT3: now also IC15A.O, IC16A.I0; no longer IC4A.O, IC5A.I0
- net NEXT4: now also IC16A.O, IC17A.I0; no longer IC5A.O, IC6A.I0
- net NEXT5: now also IC17A.O, IC18A.I0; no longer IC6A.O, IC7A.I0
- net NEXT6: now also IC18A.O, IC19A.CLK; no longer IC1A.CLK, IC7A.O
- net STEP1: now also IC13A.I1, IC7G$1.Q; no longer IC2A.I1, IC8G$1.Q
- net STEP2: now also IC14A.I1, IC8G$1.Q; no longer IC3A.I1, IC9G$1.Q
- net STEP3: now also IC15A.I1, IC9G$1.Q; no longer IC10G$1.Q, IC4A.I1
- net STEP4: now also IC10G$1.Q, IC16A.I1; no longer IC11G$1.Q, IC5A.I1
- net STEP5: now also IC11G$1.Q, IC17A.I1; no longer IC12G$1.Q, IC6A.I1
- net STEP6: now also IC12G$1.Q, IC18A.I1; no longer IC13G$1.Q, IC7A.I1
- net VAL1: now also IC1A.I1, JP1.2; no longer IC14A.I1, JP2.2
- net VAL2: now also IC2A.I1, JP2.2; no longer IC15A.I1, JP2.3
- net VAL3: now also IC3A.I1, JP3.2; no longer IC16A.I1, JP2.4
- net VAL4: now also IC4A.I1, JP4.2; no longer IC17A.I1, JP2.5
- net VAL5: now also IC5A.I1, JP5.2; no longer IC18A.I1, JP2.6
- net VAL6: now also IC6A.I1, JP6.2; no longer IC19A.I1, JP2.7
- net VCC: now also IC19P.VDD, JP3.1, JP4.1, JP5.1, JP6.1, JP7.1; no longer IC1P.VDD
Other:
- moved on the sheet: C1, C10, C11, C12, C13, C14, C15, C16, C17, C18, C19, C2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

Commit message: rework of cabling for reset, exec, power, and key-up detection
Parts:
- added C21, C22: 0.1uF, resistor:C-USC0603
- added IC22: 74AHC1G08DBV, 74xx-little-us:74AHC1G08DBV
- added IC23: 74LVC1G14DBV, 74xx-little-us:74LVC1G14DBV
- JP6, JP7: device custom-pinhead:PINHD-1X4 -> custom-pinhead:PINHD-1X5
Connections:
- removed net !MCLK: IC1A.I0, IC2A.I0, IC3A.I0, IC4A.I0, IC5A.I0, IC6A.I0, JP7.3
- new net !KEY: IC1A.I0, IC2A.I0, IC3A.I0, IC4A.I0, IC5A.I0, IC6A.I0, JP7.4
- new net !RST_OUT: IC23A.O, JP6.4
- new net EXEC: IC22A.I1, JP7.3
- new net N$7: IC22A.O, JP6.3
- net GND: now also C21.2, C22.2, JP6.5, JP7.5; no longer JP6.4, JP7.4
- net RESET: now also IC23A.I
- net SEL6: now also IC22A.I0; no longer JP6.3
- net VCC: now also C21.1, C22.1
Other:
- moved on the sheet: IC20, IC21, R2

Commit message: rework design: reduced logic to minimum, added 555 timer for debouncing moved encoder connector to top edge of board for easy routing of cabling, changed the pulse-generator connector back to 4-pin for easy cabling, cleaned up all the core routing and run detailed drc
Parts:
- removed IC1, IC2, IC3, IC4, IC5, IC6: 74AHC1G08DBV, 74xx-little-us:74AHC1G08DBV
- removed IC13: 74AHC1G32DBV, 74xx-little-us:74AHC1G32DBV
- added C23: 0.1uF, resistor:C-USC0603
- added D1, D2: MBR0520LT, diode:MBR0520LT
- added IC24: 74LVC1G14DBV, 74xx-little-us:74LVC1G14DBV
- added IC25: 74LVC1G17DBV, 74xx-little-us:74LVC1G17DBV
- added IC26: 74AHC1G08DBV, 74xx-little-us:74AHC1G08DBV
- added R3: 100K, resistor:R-US_R0805
- added R4: 47K, resistor:R-US_R0805
- C22: value 0.1uF -> 10uF; device resistor:C-USC0603 -> resistor:C-USC0805
- IC10, IC11, IC12, IC7, IC8, IC9: value 741G175 -> 74AHC1G08DBV; device witch-e:741G175 -> 74xx-little-us:74AHC1G08DBV
- IC20: value 74LVC1G14DBV -> 74LVC1G17DBV; device 74xx-little-us:74LVC1G14DBV -> 74xx-little-us:74LVC1G17DBV
- IC23: value 74LVC1G14DBV -> NE555D; device 74xx-little-us:74LVC1G14DBV -> adafruit:NE555D
- JP6: device custom-pinhead:PINHD-1X5 -> custom-pinhead:PINHD-1X4
- R1: value (none) -> 270R
- R2: value (none) -> 1K
Connections:
- net NEXT2 renamed CLK1
- net NEXT3 renamed CLK2
- net NEXT4 renamed CLK3
- net NEXT5 renamed CLK4
- removed net !RESET: IC10G$1.!CLR, IC11G$1.!CLR, IC12G$1.!CLR, IC20A.O, IC7G$1.!CLR, IC8G$1.!CLR, IC9G$1.!CLR
- removed net !RST_OUT: IC23A.O, JP6.4
- removed net N$1: IC2A.O, IC8G$1.CLK
- removed net N$2: IC1A.O, IC7G$1.CLK
- removed net N$3: IC3A.O, IC9G$1.CLK
- removed net N$4: IC10G$1.CLK, IC4A.O
- removed net N$5: IC11G$1.CLK, IC5A.O
- removed net N$6: IC12G$1.CLK, IC6A.O
- removed net NEXT1: IC13A.O, IC14A.I0
- removed net NEXT6: IC18A.O, IC19A.CLK
- new net !KEY_IN: D1.C, D2.C, JP7.4
- new net CLK5: IC18A.O, IC26A.I1
- new net N$10: D1.A, IC23.TR, R3.1
- new net N$11: IC23.Q, IC24A.I
- new net N$12: IC25A.I, JP7.3
- new net N$13: C23.1, IC20A.I, R2.1
- new net N$14: IC26A.O, R2.2
- new net N$8: IC19A.CLK, IC20A.O
- new net N$9: C22.1, D2.A, IC23.DIS, IC23.THR, R4.1
- net !KEY: now also IC24A.O, IC26A.I0; no longer IC1A.I0, IC2A.I0, IC3A.I0, IC4A.I0, IC5A.I0, IC6A.I0, JP7.4
- net EXEC: now also IC25A.O; no longer JP7.3
- net GND: now also C23.2, IC23.GND, JP6.4; no longer IC13A.I0, JP6.5, R2.1
- net RESET: no longer IC20A.I, IC23A.I, R2.2
- net SEL1: now also IC7A.I1; no longer IC7G$1.D
- net SEL2: now also IC8A.I1; no longer IC8G$1.D
- net SEL3: now also IC9A.I1; no longer IC9G$1.D
- net SEL4: now also IC10A.I1; no longer IC10G$1.D
- net SEL5: now also IC11A.I1; no longer IC11G$1.D
- net SEL6: now also IC12A.I1; no longer IC12G$1.D
- net STEP1: now also IC14A.I0, IC7A.O; no longer IC13A.I1, IC7G$1.Q
- net STEP2: now also IC8A.O; no longer IC8G$1.Q
- net STEP3: now also IC9A.O; no longer IC9G$1.Q
- net STEP4: now also IC10A.O; no longer IC10G$1.Q
- net STEP5: now also IC11A.O; no longer IC11G$1.Q
- net STEP6: now also IC12A.O; no longer IC12G$1.Q
- net VAL1: now also IC7A.I0; no longer IC1A.I1
- net VAL2: now also IC8A.I0; no longer IC2A.I1
- net VAL3: now also IC9A.I0; no longer IC3A.I1
- net VAL4: now also IC10A.I0; no longer IC4A.I1
- net VAL5: now also IC11A.I0; no longer IC5A.I1
- net VAL6: now also IC12A.I0; no longer IC6A.I1
- net VCC: now also IC23.R, IC23.V+, R3.2, R4.2; no longer C22.1
Other:
- note added: "R3"
- moved on the sheet: C1, C10, C11, C12, C13, C14, C15, C16, C17, C18, C19, C2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
