File: block-designs/witch-phase2/pulse-generator/pulse-generator.sch (EAGLE design)
At the start: 92 parts, among them IC1 74LVC1G08DBV, IC10 74LVC1G08DBV, IC11 741G175, IC12 74LVC1G08DBV, IC13 741G175, IC14 741G175, IC15 741G175, IC16 74LVC1G04DBV, IC17 741G175, IC18 74LVC1G04DBV, IC19 74LVC1G04DBV, IC2 741G175, IC20 NE555D, IC21 74LVC1G17DBV, IC22 74LVC1G17DBV, IC23 74LVC1G17DBV, IC24 74LVC1G04DBV, IC3 741G175, IC4 741G175, IC5 74LVC1G04DBV, IC6 74LVC1G08DBV, IC7 741G175, IC8 74LVC1G08DBV, IC9 74LVC1G08DBV, J1 POWER_JACKPTH, Q1 MMBT2907ALT1SMD, Q2 MMBT2222A, Q3 MMBT2222A, Q4 MMBT2222A, Q5 MMBT2222A, Q6 MMBT2222A

Commit message: routing tweaks for LEDs
Parts:
- C14, C15, C16: value 10uF -> 0.1uF
- C18, C19: value (none) -> 0.1uF
- C21, C23, C4: value 0.1uF -> 10uF
- C26, C27: value 0.1uF -> (none)
- IC11, IC13: value 741G175 -> 74LVC1G08DBV; device witch-e:741G175 -> 74xx-little-us:74LVC1G08DBV
- IC12, IC8: value 74LVC1G08DBV -> 741G175; device 74xx-little-us:74LVC1G08DBV -> witch-e:741G175
- IC16, IC18: value 74LVC1G04DBV -> 741G175; device 74xx-little-us:74LVC1G04DBV -> witch-e:741G175
- IC17, IC7: value 741G175 -> 74LVC1G04DBV; device witch-e:741G175 -> 74xx-little-us:74LVC1G04DBV
- IC20: value NE555D -> 74LVC1G04DBV; device adafruit:NE555D -> 74xx-little-us:74LVC1G04DBV
- IC21: value 74LVC1G17DBV -> NE555D; device 74xx-little-us:74LVC1G17DBV -> adafruit:NE555D
- IC24: value 74LVC1G04DBV -> 74LVC1G17DBV; device 74xx-little-us:74LVC1G04DBV -> 74xx-little-us:74LVC1G17DBV
- JP1: device pinhead:PINHD-1X11 -> pinhead:PINHD-1X4
- JP2: device pinhead:PINHD-1X2 -> pinhead:PINHD-1X11
- JP3: device pinhead:PINHD-1X4 -> pinhead:PINHD-1X2
- Q1: value MMBT2907ALT1SMD -> MMBT2222A; device transistor-pnp:MMBT2907ALT1SMD -> SparkFun-DiscreteSemi:TRANSISTOR_NPNMMBT2222A
- Q6: value MMBT2222A -> MMBT2907ALT1SMD; device SparkFun-DiscreteSemi:TRANSISTOR_NPNMMBT2222A -> transistor-pnp:MMBT2907ALT1SMD
- R1, R14, R7: value 270 -> 1K
- R10: value (none) -> 270
- R11: value (none) -> 8.2K
- R12: value (none) -> 33K
- R13: value 1K -> 10k
- R15: value 1K -> 100k
- R16, R18: value 270 -> (none)
- R17, R19: value 1K -> (none)
- R2: value 8.2K -> 270
- R3: value 33K -> 1K
- R4: value 10k -> 270
- R6: value 100k -> 270
- R8: value 1K -> 270
- R9: value (none) -> 1K
Connections:
- removed net N$11 (its old number): IC13G$1.Q, IC14G$1.D
- removed net N$37 (its old number): LED6.C, Q6.C
- removed net N$5 (its old number): Q1.B, R8.1
- removed net N$7 (its old number): LED1.A, R7.2
- new net N$13: LED1.C, Q1.C
- new net N$17: IC15G$1.Q, IC16G$1.D
- new net N$38: Q5.B, R9.1
- new net N$39: LED5.A, R10.2
- net !CDONE: now also IC13A.I1, IC17A.O; no longer IC12A.I1, IC16A.O
- net !MCLK: now also IC11A.I1, IC16G$1.CLK, IC20A.O, JP2.2; no longer IC10A.I1, IC14G$1.CLK, IC19A.O, JP1.2
- net !RST: now also IC12G$1.!CLR, IC16G$1.!CLR, IC18G$1.!CLR, IC24G$1.O, IC8G$1.!CLR, JP2.1, JP2.8; no longer IC11G$1.!CLR, IC13G$1.!CLR, IC17G$1.!CLR, IC23G$1.O, IC7G$1.!CLR, JP1.1, JP1.8
- net 10A_PULSE: now also IC7A.I, JP1.2, JP2.9, R1.2; no longer IC24A.I, JP1.9, JP3.2, R15.2
- net 9A_PULSE: now also JP2.10; no longer JP1.10
- net ADD/COMP: now also IC23G$1.O, JP2.7; no longer IC22G$1.O, JP1.7
- net CARRY_DONE: now also IC14G$1.CLK, JP2.4; no longer IC13G$1.CLK, JP1.4
- net CARRY_OE: now also IC10A.I1, IC13A.O, JP2.3, R7.2; no longer IC12A.O, IC9A.I1, JP1.3, R19.2
- net CARRY_PULSE: now also IC10A.O, JP2.6, R5.2; no longer IC9A.O, JP1.6, R13.2
- net CDONE: now also IC16G$1.Q, IC17A.I, R9.2; no longer IC15G$1.Q, IC16A.I, R21.2
- net CLR: now also IC22G$1.O, JP2.11; no longer IC21G$1.O, JP1.11
- net GND: now also IC21.GND, JP1.4, JP3.2, LED6.C, Q1.E; no longer IC20.GND, JP2.2, JP3.4, LED1.C, Q6.E
- net MCLK: now also IC18G$1.CLK, IC20A.I, IC21.Q, R21.2; no longer IC17G$1.CLK, IC19A.I, IC20.Q, R8.2
- net N$1: now also IC18G$1.D, IC19A.O; no longer IC17G$1.D, IC18A.O
- net N$12: now also IC8G$1.Q; no longer IC7G$1.Q
- net N$15: now also IC12G$1.Q, IC13A.I0; no longer IC11G$1.Q, IC12A.I0
- net N$16: now also IC11A.O, IC12G$1.CLK; no longer IC10A.O, IC11G$1.CLK
- net N$19: now also C23.1, IC24G$1.I, R13.2; no longer C16.1, IC23G$1.I, R4.2
- net N$2: now also C21.1, IC21.THR, IC21.TR, R11.1, R12.1; no longer C14.1, IC20.THR, IC20.TR, R2.1, R3.1
- net N$20: now also R13.1, R15.1; no longer R4.1, R6.1
- net N$21: now also C26.1, IC22G$1.I, R17.2; no longer C18.1, IC21G$1.I, R10.2
- net N$22: now also R16.1, R17.1; no longer R10.1, R9.1
- net N$23: now also IC7A.O, IC8G$1.CLK; no longer IC24A.O, IC7G$1.CLK
- net N$24: now also Q3.B, R5.1; no longer Q2.B, R13.1
- net N$25: now also LED3.A, R6.2; no longer LED2.A, R1.2
- net N$26: now also Q1.B, R1.1; no longer Q3.B, R15.1
- net N$28: now also LED1.A, R2.2; no longer LED3.A, R14.2
- net N$29: now also C27.1, IC23G$1.I, R19.2; no longer C19.1, IC22G$1.I, R12.2
- net N$3: now also IC21.DIS, R12.2, R14.1; no longer IC20.DIS, R3.2, R5.1
- net N$30: now also R18.1, R19.1; no longer R11.1, R12.1
- net N$32: now also Q2.B, R3.1; no longer Q4.B, R17.1
- net N$33: now also LED2.A, R4.2; no longer LED4.A, R16.2
- net N$35: now also Q4.B, R7.1; no longer Q5.B, R19.1
- net N$36: now also LED4.A, R8.2; no longer LED5.A, R18.2
- net N$4: now also R11.2; no longer R2.2
- net N$6: now also Q6.C, R20.1; no longer Q1.C, R7.1
- net N$9: now also IC10A.I0, IC9A.O; no longer IC8A.O, IC9A.I0
- net TCLK: now also IC18G$1.Q, IC19A.I, IC9A.I1; no longer IC17G$1.Q, IC18A.I, IC8A.I1
- net TDONE: now also IC11A.I0, IC9A.I0, R3.2; no longer IC10A.I0, IC8A.I0, R17.2
- net VCC: now also C14.1, C16.1, C18.1, C19.1, IC12G$1.D, IC14G$1.D, IC21.R, IC21.V+, IC8G$1.D, JP1.1, Q6.E, R10.1, R14.2, R15.2, R16.2, R18.2, R2.1, R4.1, R6.1, R8.1; no longer C21.1, C23.1, C26.1, C27.1, IC11G$1.D, IC13G$1.D, IC20.R, IC20.V+, IC7G$1.D, JP2.1, Q1.E, R1.1, R11.2, R14.1, R16.1, R18.1, R20.1, R5.2, R6.2, R9.2
- net ZC: now also JP1.3; no longer JP3.3

Commit message: add new connectors for input system and bug fixes from earlier prototype
Parts:
- removed C25: 0.1uF, resistor:C-USC0805
- removed C26, C27: (no value), resistor:C-USC0805
- removed IC24: 74LVC1G17DBV, 74xx-little-us:74LVC1G17DBV
- removed J1: POWER_JACKPTH, SparkFun-Connectors:POWER_JACKPTH
- removed R19: (no value), resistor:R-US_R0805
- removed R20: 270, resistor:R-US_R0805
- removed R21: 1K, resistor:R-US_R0805
- removed S2: (no value), SparkFun-Electromechanical:TAC_SWITCHPTH
- removed S3, S4: (no value), SparkFun-Electromechanical:SWITCH-SPDTPTH
- added D1, D2, D3, D4: MBR0520LT, diode:MBR0520LT
- added JP4: (no value), pinhead:PINHD-1X4
- added JP5: (no value), custom-pinhead:PINHD-1X6
- C1: value 10uF -> 0.1uF
- C10, C11, C12, C14, C15, C16, C17, C18, C19, C20, C22, C24, C3, C5, C6, C8, C9: device resistor:C-USC0805 -> resistor:C-USC0603
- C2: value 0.1uF -> 10uF
- C21, C23: value 10uF -> 0.1uF; device resistor:C-USC0805 -> resistor:C-USC0603
- IC1: value 74LVC1G08DBV -> 74LVC1G17DBV; device 74xx-little-us:74LVC1G08DBV -> 74xx-little-us:74LVC1G17DBV
- IC13, IC9: value 74LVC1G08DBV -> 741G175; device 74xx-little-us:74LVC1G08DBV -> witch-e:741G175
- IC18: value 741G175 -> 74LVC1G04DBV; device witch-e:741G175 -> 74xx-little-us:74LVC1G04DBV
- IC19: value 74LVC1G04DBV -> 74LVC1G08DBV; device 74xx-little-us:74LVC1G04DBV -> 74xx-little-us:74LVC1G08DBV
- IC2, IC3: value 741G175 -> 74LVC1G17DBV; device witch-e:741G175 -> 74xx-little-us:74LVC1G17DBV
- IC21: value NE555D -> 74LVC1G08DBV; device adafruit:NE555D -> 74xx-little-us:74LVC1G08DBV
- IC22: value 74LVC1G17DBV -> 741G175; device 74xx-little-us:74LVC1G17DBV -> witch-e:741G175
- IC23: value 74LVC1G17DBV -> 74LVC1G08DBV; device 74xx-little-us:74LVC1G17DBV -> 74xx-little-us:74LVC1G08DBV
- IC4: value 741G175 -> NE555D; device witch-e:741G175 -> adafruit:NE555D
- IC5: value 74LVC1G04DBV -> 741G175; device 74xx-little-us:74LVC1G04DBV -> witch-e:741G175
- IC6: value 74LVC1G08DBV -> 74LVC1G04DBV; device 74xx-little-us:74LVC1G08DBV -> 74xx-little-us:74LVC1G04DBV
- JP1: device pinhead:PINHD-1X4 -> pinhead:PINHD-1X2
- JP2: device pinhead:PINHD-1X11 -> pinhead:PINHD-1X4
- JP3: device pinhead:PINHD-1X2 -> pinhead:PINHD-1X11
- R11: value 8.2K -> 270
- R12: value 33K -> 8.2K
- R13: value 10k -> 1K
- R15: value 100k -> 33K
- R16, R18: value (none) -> 270
- R17: value (none) -> 1K
- R2, R8: value 270 -> 1K
- R3: value 1K -> 270
- R5, R7: value 1K -> 100k
- R6: value 270 -> 100k
Connections:
- removed net N$12: IC1A.I1, IC8G$1.Q
- removed net N$14: IC3G$1.Q, IC4G$1.D
- removed net N$20: R13.1, R15.1, S2.3, S2.4
- removed net N$21: C26.1, IC22G$1.I, R17.2
- removed net N$22: R16.1, R17.1, S3.P
- removed net N$29: C27.1, IC23G$1.I, R19.2
- removed net N$30: R18.1, R19.1, S4.P
- new net !EXE: C1.1, IC3G$1.I, JP4.3, R7.1
- new net CARRY_INIT: IC11A.I0, IC12G$1.Q, IC14G$1.D
- new net FOUR: JP5.6
- new net N$18: D1.C, D2.C, IC1G$1.I, R5.2
- new net ONE: D3.A, JP5.3
- new net THREE: D2.A, D4.A, JP5.5
- new net TWO: D1.A, JP5.4
- new net ZERO: JP5.2
- net !CDONE: now also IC18A.O, IC21A.I1; no longer IC13A.I1, IC17A.O
- net !MCLK: now also IC12G$1.CLK, IC13G$1.CLK, IC14G$1.CLK, IC7A.O, JP3.2; no longer IC15G$1.CLK, IC20A.O, IC3G$1.CLK, IC4G$1.CLK, JP2.2
- net !RST: now also IC13G$1.!CLR, IC22G$1.!CLR, IC3G$1.O, IC5G$1.!CLR, IC9G$1.!CLR, JP3.1, JP3.8; no longer IC18G$1.!CLR, IC24G$1.O, IC2G$1.!CLR, IC3G$1.!CLR, IC4G$1.!CLR, JP2.1, JP2.8
- net !TDONE: now also IC17A.O, IC19A.I0; no longer IC5A.O, IC6A.I0
- net 10A_PULSE: now also IC19A.O, IC20A.I, JP2.2, JP3.9; no longer IC1A.I0, IC6A.O, IC7A.I, JP1.2, JP2.9
- net 9A_PULSE: now also IC22G$1.Q, JP3.10; no longer IC1A.O, JP2.10
- net ADD/COMP: now also IC1G$1.O, JP3.7; no longer IC23G$1.O, JP2.7
- net CARRY_DONE: now also IC9G$1.CLK, JP3.4; no longer IC14G$1.CLK, JP2.4
- net CARRY_OE: now also IC21A.O, IC23A.I1, JP3.3, R9.2; no longer IC10A.I1, IC13A.O, JP2.3, R7.2
- net CARRY_PULSE: now also IC23A.O, JP3.6, R8.2; no longer IC10A.O, JP2.6, R5.2
- net CDONE: now also IC18A.I, JP4.2, R13.2; no longer IC17A.I, R9.2
- net CLR: now also IC2G$1.O, JP3.11; no longer IC22G$1.O, JP2.11
- net GND: now also IC4.GND, JP1.2, JP2.4, JP4.4, JP5.1, R5.1, R6.1; no longer C25.2, C26.2, C27.2, IC21.GND, J1.GND, J1.GNDBREAK, JP1.4, JP3.2, S2.1, S2.2, S3.S, S4.S
- net MCLK: now also IC4.Q, IC5G$1.CLK, IC7A.I, R17.2; no longer IC18G$1.CLK, IC20A.I, IC21.Q, R21.2
- net N$1: now also IC5G$1.D, IC6A.O; no longer IC18G$1.D, IC19A.O
- net N$11: now also IC13G$1.D, IC9G$1.Q; no longer IC14G$1.Q, IC15G$1.D
- net N$15: now also IC15G$1.Q, IC21A.I0; no longer IC12G$1.Q, IC13A.I0
- net N$16: now also IC15G$1.CLK; no longer IC12G$1.CLK
- net N$17: now also IC13G$1.Q; no longer IC15G$1.Q
- net N$19: now also D3.C, D4.C, IC2G$1.I, R6.2; no longer C23.1, IC24G$1.I, R13.2
- net N$2: now also C2.1, IC4.THR, IC4.TR, R15.1; no longer C21.1, IC21.THR, IC21.TR, R11.1
- net N$23: now also IC20A.O, IC22G$1.CLK; no longer IC7A.O, IC8G$1.CLK
- net N$24: now also R8.1; no longer R5.1
- net N$25: now also R10.2; no longer R6.2
- net N$28: now also R3.2; no longer R2.2
- net N$3: now also IC4.DIS, R15.2; no longer IC21.DIS, R12.2
- net N$32: now also R2.1; no longer R3.1
- net N$35: now also R9.1; no longer R7.1
- net N$36: now also R11.2; no longer R8.2
- net N$38: now also R13.1; no longer R9.1
- net N$39: now also R16.2; no longer R10.2
- net N$4: now also R12.2; no longer R11.2
- net N$5: now also R17.1; no longer R21.1
- net N$6: now also R18.1; no longer R20.1
- net N$7: now also R18.2; no longer R20.2
- net N$8: now also IC12G$1.D, IC8G$1.Q; no longer IC2G$1.Q, IC3G$1.D
- net N$9: now also IC10A.O, IC23A.I0; no longer IC10A.I0, IC9A.O
- net TCLK: now also IC10A.I1, IC19A.I1, IC5G$1.Q, IC6A.I; no longer IC18G$1.Q, IC19A.I, IC6A.I1, IC9A.I1
- net TDONE: now also IC10A.I0, IC14G$1.Q, IC17A.I, R2.2; no longer IC11A.I0, IC4G$1.Q, IC5A.I, IC9A.I0, R3.2
- net VCC: now also C21.1, C23.1, IC15G$1.D, IC22G$1.D, IC4.R, IC4.V+, IC9G$1.D, JP2.1, JP4.1, R11.1, R16.1, R3.1, R7.2; no longer C1.1, C2.1, C25.1, IC12G$1.D, IC14G$1.D, IC21.R, IC21.V+, IC2G$1.D, J1.PWR, JP3.1, R15.2, R16.2, R18.2, R2.1, R6.1, R8.1
- net ZC: now also IC8G$1.CLK, JP2.3; no longer IC2G$1.CLK, JP1.3
Other:
- moved on the sheet: C1, C10, C11, C12, C13, C14, C15, C16, C17, C19, C2, C20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
